File: Euro-LFO.kicad_pcb (KiCad board)
At the start: 2 copper layers, 56.2 x 128.5 mm, 30 parts, among them J1 Conn_02x05_Odd_Even, Q1 NPN, U1 TL074

Commit message: updated
Parts:
- added C6: 10 µF 25 V X5R, Capacitor_SMD:C_0805_2012Metric, F.Cu at (138.0, 85.5)
- added C7: 10 µF 25 V X5R, Capacitor_SMD:C_0805_2012Metric, F.Cu at (130.0, 81.0)
- added D4: SS14 (40 V 1 A Schottky), Diode_SMD:D_SMA, F.Cu at (144.0, 122.0)
- added D5: SS14 (40 V 1 A Schottky), Diode_SMD:D_SMA, F.Cu at (129.0, 122.0)
- added R23: 10 Ω 0805, Resistor_SMD:R_0805_2012Metric, F.Cu at (144.0, 114.0)
- added R24: 10 Ω 0805, Resistor_SMD:R_0805_2012Metric, F.Cu at (129.0, 114.1)
- C1, C2: value 47n -> 100 nF 50 V X7R
- C3: value 47n -> 00 nF 50 V X7R
- D1, D2: value 1N914 -> 1N4148W
- D3: value LED -> 3 mm LED
- INV-OUT1, PWM-OUT1, TRI-OUT1: value ~ -> 3.5 mm mono jack, Thonkiconn PJ398SM
- J1: value Conn_02x05_Odd_Even -> 2×5 2.54 mm shrouded IDC box header; footprint Connector_PinHeader_2.54mm:PinHeader_2x05_P2.54mm_Vertical -> Connector_IDC:IDC-Header_2x05_P2.54mm_Vertical
- OFFSET1: value 100K -> 100 kΩ B (linear), centre-detent if available
- Q1: value NPN -> MMBT3904
- R1: value 150K -> 150 kΩ 0805 1%
- R14, R4: value 4K7 -> 4.7 kΩ 0805 1%
- R16, R18, R19, R21, R22, R5: value 100K -> 100 kΩ 0805 1%
- R17, R20: value 1K -> 1 kΩ 0805 1%
- R2: value 2K2 -> 2.2 kΩ 0805 1%
- R3: value 1K -> 1 kΩ 0805
- R6: value 10K -> 10 kΩ 0805 1%
- RANGE1: value 100K -> 100 kΩ A (audio) for smoother level control (B works)
- RATE1: value 100K -> 100 kΩ Alpha 9 mm vertical - taper B (or reverse‑log for feel)
- SHAPE1: value 500K -> 500 kΩ B (linear)
- U1: value TL074 -> TL074CDR
- moved R21 59.7 mm to (135.0, 71.1), turned to -90 degrees
- moved R22 57.4 mm to (130.0, 76.1), turned to -90 degrees
- moved R20 57.1 mm to (138.0, 71.1), turned to 90 degrees
- moved TRI-OUT1 48.4 mm to (107.0, 120.6)
- moved R19 45.4 mm to (141.0, 70.9), turned to 90 degrees
- moved R18 43.4 mm to (144.0, 75.9), turned to 90 degrees
- moved C1 42.1 mm to (141.0, 90.5), turned to 90 degrees
- moved R14 41.6 mm to (132.0, 95.5)
- moved R6 37.3 mm to (144.0, 85.6), turned to -90 degrees
- moved R16 36.2 mm to (144.0, 70.9)
- moved J1 36.0 mm to (137.5, 124.0), turned to 180 degrees
- moved Q1 34.6 mm to (136.1, 90.9), turned to -90 degrees
- moved D2 33.4 mm to (136.0, 65.0), turned to -90 degrees
- moved R4 32.8 mm to (144.0, 65.0)
- moved R5 31.3 mm to (141.0, 85.5), turned to -90 degrees
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Connections:
- net Net-(D3-A) renamed /LED_A
- net Net-(INV-OUT1-PadT) renamed /INV-OUT-A
- net Net-(R17-Pad1) renamed /TRI-OUT-A
- J1 pad 1: +12V -> Net-(D5-K)
- J1 pad 10: -12V -> Net-(D4-A)
- J1 pad 2: +12V -> Net-(D5-K)
- J1 pad 9: -12V -> Net-(D4-A)
- Q1 pad 1: +12V -> Net-(Q1-B)
- Q1 pad 2: Net-(Q1-B) -> Net-(Q1-E)
- Q1 pad 3: Net-(Q1-E) -> +12V
Other:
- board size 56.2 x 128.5 mm -> 81 x 128.5 mm

Commit message: added pin headers
Parts:
- added J3: Conn_01x07_Socket, Connector_PinHeader_2.54mm:PinHeader_1x07_P2.54mm_Vertical, F.Cu at (128.5, 56.5)
- added J4: Conn_01x07_Pin, Connector_PinHeader_2.54mm:PinHeader_1x07_P2.54mm_Vertical, F.Cu at (120.5, 56.5)
- added J5: Conn_01x07_Socket, Connector_PinHeader_2.54mm:PinHeader_1x07_P2.54mm_Vertical, F.Cu at (145.0, 89.8)
- added J6: Conn_01x07_Pin, Connector_PinHeader_2.54mm:PinHeader_1x07_P2.54mm_Vertical, F.Cu at (103.5, 89.8)
- moved R4 32.5 mm to (119.5, 43.6)
- moved D1 24.6 mm to (108.5, 62.5), turned to 180 degrees
- moved D2 21.1 mm to (115.0, 62.5), turned to 180 degrees
- moved Q1 10.2 mm to (135.0, 101.1)
- moved C1 9.62 mm to (139.5, 100.0)
- moved R20 9.18 mm to (135.0, 62.4), turned to -90 degrees
- moved R14 6.93 mm to (129.9, 102.1)
- moved C3 5.72 mm to (130.9, 96.1)
- moved R1 5.42 mm to (130.0, 90.8)
- moved R2 5.42 mm to (133.0, 90.9)
- moved R3 5.42 mm to (136.0, 90.9)
- moved R21 4.50 mm to (135.0, 66.6)
- moved R19 2.08 mm to (139.0, 71.5), turned to 180 degrees
- moved R17 1.12 mm to (133.0, 71.6)
- moved R16 0.71 mm to (143.5, 70.4)
Connections:
- C1 pad 2: Net-(Q1-B) -> /RNG_3_I
- D3 pad 1: GND -> /GND_O
- D3 pad 2: /LED_A -> /LED_O
- INV-OUT1 pad S: GND -> /GND_O
- OFFSET1 pad 1: +12V -> /+12_O
- OFFSET1 pad 2: Net-(OFFSET1-Pad2) -> /OFF_O
- OFFSET1 pad 3: -12V -> /-12_O
- PWM-OUT1 pad S: GND -> /GND_O
- PWM-OUT1 pad T: Net-(PWM-OUT1-PadT) -> /PWM_O
- Q1 pad 1: Net-(Q1-B) -> /RNG_3_I
- R1 pad 2: Net-(R1-Pad2) -> /U!A_I
- R14 pad 2: /LED_A -> /LED_I
- R16 pad 2: Net-(OFFSET1-Pad2) -> /OFF_I
- R17 pad 1: /TRI-OUT-A -> /TRI_I
- R19 pad 2: Net-(R19-Pad2) -> /RNG_2_I
- R2 pad 1: Net-(PWM-OUT1-PadT) -> /PWM_I
- R2 pad 2: Net-(R1-Pad2) -> /U!A_I
- R20 pad 1: /INV-OUT-A -> /INV_I
- R3 pad 2: Net-(PWM-OUT1-PadT) -> /PWM_I
- R4 pad 1: GND -> /GND_O
- R5 pad 1: Net-(Q1-B) -> /RNG_3_I
- R6 pad 2: Net-(R6-Pad2) -> /SHP_I
- RANGE1 pad 1: Net-(Q1-B) -> /GND_O
- RANGE1 pad 2: Net-(R19-Pad2) -> /RNG_2_O
- RANGE1 pad 3: GND -> /RNG_3_O
- RATE1 pad 1: Net-(R1-Pad2) -> /U1A_O
- SHAPE1 pad 2: Net-(R6-Pad2) -> /SHP_O
- TRI-OUT1 pad S: GND -> /GND_O
- TRI-OUT1 pad T: /TRI-OUT-A -> /TRI_O
- U1 pad 1: Net-(R1-Pad2) -> /U!A_I
- U1 pad 7: Net-(Q1-B) -> /RNG_3_I

Commit message: work in progress
Parts:
- moved R6 8.45 mm to (137.1, 90.5)
- moved C6 5.88 mm to (132.1, 86.0)
- moved R22 5.84 mm to (133.6, 71.5)
- moved R1 5.67 mm to (127.1, 85.9)
- moved R5 5.40 mm to (135.6, 86.1)
- moved C1 4.21 mm to (137.1, 96.6)
- moved C2 4.20 mm to (141.1, 84.0)
- moved C7 3.51 mm to (127.1, 79.0)
- moved R2 3.37 mm to (129.6, 90.9)
- moved R18 2.93 mm to (141.1, 76.5)
- moved D4 2.87 mm to (141.1, 122.0)
- moved J5 2.87 mm to (142.1, 89.9)
- moved Q1 2.87 mm to (132.1, 101.1), turned to 0 degrees
- moved R16 2.87 mm to (140.6, 70.4)
- moved R17 2.87 mm to (130.1, 71.6)
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Connections:
- J5 pad 5: unconnected-(J5-Pin_5-Pad5) -> /U1A_I
- J6 pad 5: unconnected-(J6-Pin_5-Pad5) -> /U1A_O
- R1 pad 2: /U!A_I -> /U1A_I
- R2 pad 2: /U!A_I -> /U1A_I
- U1 pad 1: /U!A_I -> /U1A_I
Other:
- board size 81 x 128.5 mm -> 65.1 x 128.5 mm

Commit message: Sorting out cross board connections
Connections:
- J5 pad 1: +12V -> /U1A_I
- J5 pad 2: /OFF_I -> +12V
- J5 pad 3: /RNG_3_I -> /OFF_I
- J5 pad 4: /RNG_2_I -> -12V
- J5 pad 5: /U1A_I -> /RNG_3_I
- J5 pad 6: unconnected-(J5-Pin_6-Pad6) -> /RNG_2_I
- J5 pad 7: -12V -> unconnected-(J5-Pin_7-Pad7)
- J6 pad 1: /+12_O -> /U1A_O
- J6 pad 2: /OFF_O -> /+12_O
- J6 pad 3: /RNG_3_O -> /OFF_O
- J6 pad 4: /RNG_2_O -> /-12_O
- J6 pad 5: /U1A_O -> /RNG_3_O
- J6 pad 6: unconnected-(J6-Pin_6-Pad6) -> /RNG_2_O
- J6 pad 7: /-12_O -> unconnected-(J6-Pin_7-Pad7)
Changed lines of the file:
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@@
 			(layers "*.Cu" "*.Mask")
 			(remove_unused_layers no)
-			(net "/+12_O")
+			(net "/U1A_O")
 			(pinfunction "Pin_1_1")
 			(pintype "passive")
@@
 			(layers "*.Cu" "*.Mask")
 			(remove_unused_layers no)
-			(net "/OFF_O")
+			(net "/+12_O")
 			(pinfunction "Pin_2_2")
 			(pintype "passive")
@@
 			(layers "*.Cu" "*.Mask")
 			(remove_unused_layers no)
-			(net "/RNG_3_O")
+			(net "/OFF_O")
 			(pinfunction "Pin_3_3")
 			(pintype "passive")
@@
 			(layers "*.Cu" "*.Mask")
 			(remove_unused_layers no)
-			(net "/RNG_2_O")
+			(net "/-12_O")
 			(pinfunction "Pin_4_4")
 			(pintype "passive")
@@
 			(layers "*.Cu" "*.Mask")
 			(remove_unused_layers no)
-			(net "/U1A_O")
+			(net "/RNG_3_O")
 			(pinfunction "Pin_5_5")
 			(pintype "passive")
@@
 			(layers "*.Cu" "*.Mask")
 			(remove_unused_layers no)
-			(net "unconnected-(J6-Pin_6-Pad6)")
+			(net "/RNG_2_O")
 			(pinfunction "Pin_6_6")
 			(pintype "passive")
@@
 			(layers "*.Cu" "*.Mask")
 			(remove_unused_layers no)
-			(net "/-12_O")
+			(net "unconnected-(J6-Pin_7-Pad7)")
 			(pinfunction "Pin_7_7")
 			(pintype "passive")
@@
 			(layers "*.Cu" "*.Mask")
 			(remove_unused_layers no)
-			(net "+12V")
+			(net "/U1A_I")
 			(pinfunction "Pin_1_1")
 			(pintype "passive")
@@
 			(layers "*.Cu" "*.Mask")
 			(remove_unused_layers no)
-			(net "/OFF_I")
+			(net "+12V")
 			(pinfunction "Pin_2_2")
 			(pintype "passive")
@@
 			(layers "*.Cu" "*.Mask")
 			(remove_unused_layers no)
-			(net "/RNG_3_I")
+			(net "/OFF_I")
 			(pinfunction "Pin_3_3")
 			(pintype "passive")
@@
 			(layers "*.Cu" "*.Mask")
 			(remove_unused_layers no)
-			(net "/RNG_2_I")
+			(net "-12V")
 			(pinfunction "Pin_4_4")
 			(pintype "passive")
@@
 			(layers "*.Cu" "*.Mask")
 			(remove_unused_layers no)
-			(net "/U1A_I")
+			(net "/RNG_3_I")
 			(pinfunction "Pin_5_5")
 			(pintype "passive")
@@
 			(layers "*.Cu" "*.Mask")
 			(remove_unused_layers no)
-			(net "unconnected-(J5-Pin_6-Pad6)")
+			(net "/RNG_2_I")
 			(pinfunction "Pin_6_6")
 			(pintype "passive")
@@
 			(layers "*.Cu" "*.Mask")
 			(remove_unused_layers no)
-			(net "-12V")
+			(net "unconnected-(J5-Pin_7-Pad7)")
 			(pinfunction "Pin_7_7")
 			(pintype "passive")
