File: _autosave-Euro-LFO.kicad_pcb (KiCad board)
At the start: 2 copper layers, 65.1 x 128.5 mm, 40 parts, among them J1 2×5 2.54 mm shrouded IDC box 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, J3 Conn_01x07_Socket, J4 Conn_01x07_Pin, J5 Conn_01x07_Socket, J6 Conn_01x07_Pin, Q1 MMBT3904, U1 TL074CDR

Commit message: flipped parts
Flipped parts, cleaned up edge cuts, untangled rats nest.
Connections:
- J3 pad 3: unconnected-(J3-Pin_3-Pad3) -> GND
- J3 pad 5: /PWM_I -> unconnected-(J3-Pin_5-Pad5)
- J3 pad 7: GND -> /PWM_I
- J4 pad 2: unconnected-(J4-Pin_2-Pad2) -> /INV_O
- J4 pad 3: unconnected-(J4-Pin_3-Pad3) -> /GND_O
- J4 pad 5: /PWM_O -> unconnected-(J4-Pin_5-Pad5)
- J4 pad 7: /GND_O -> /PWM_O
Routing:
- removed copper zone on B.Cu, net (none)
- removed copper zone on F.Cu, net (none)
Other:
- outline, holes or cut-outs redrawn
Changed lines of the file:
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@@
 			(layers "*.Cu" "*.Mask")
 			(remove_unused_layers no)
-			(net "unconnected-(J3-Pin_3-Pad3)")
+			(net "GND")
 			(pinfunction "Pin_3_3")
 			(pintype "passive")
@@
 			(layers "*.Cu" "*.Mask")
 			(remove_unused_layers no)
-			(net "/PWM_I")
+			(net "unconnected-(J3-Pin_5-Pad5)")
 			(pinfunction "Pin_5_5")
 			(pintype "passive")
@@
 			(layers "*.Cu" "*.Mask")
 			(remove_unused_layers no)
-			(net "GND")
+			(net "/PWM_I")
 			(pinfunction "Pin_7_7")
 			(pintype "passive")
@@
 			(layers "*.Cu" "*.Mask")
 			(remove_unused_layers no)
-			(net "unconnected-(J4-Pin_2-Pad2)")
+			(net "/INV_O")
 			(pinfunction "Pin_2_2")
 			(pintype "passive")
@@
 			(layers "*.Cu" "*.Mask")
 			(remove_unused_layers no)
-			(net "unconnected-(J4-Pin_3-Pad3)")
+			(net "/GND_O")
 			(pinfunction "Pin_3_3")
 			(pintype "passive")
@@
 			(layers "*.Cu" "*.Mask")
 			(remove_unused_layers no)
-			(net "/PWM_O")
+			(net "unconnected-(J4-Pin_5-Pad5)")
 			(pinfunction "Pin_5_5")
 			(pintype "passive")
@@
 			(layers "*.Cu" "*.Mask")
 			(remove_unused_layers no)
-			(net "/GND_O")
+			(net "/PWM_O")
 			(pinfunction "Pin_7_7")
 			(pintype "passive")
@@
 		(layer "Edge.Cuts")
 	)
-	(gr_line
-		(start 102.5 28.657257)
-		(end 105.5 28.657257)
-		(stroke
-			(width 0.5)
-			(type default)
-		)
-		(layer "Edge.Cuts")
-	)
-	(gr_line
-		(start 102.5 137.657257)
-		(end 105.5 137.657257)
-		(stroke
-			(width 0.5)
-			(type default)
-		)
-		(layer "Edge.Cuts")
-	)
-	(gr_line
-		(start 107.5 28.657257)
-		(end 110.5 28.657257)
-		(stroke
-			(width 0.5)
-			(type default)
-		)
-		(layer "Edge.Cuts")
-	)
-	(gr_line
-		(start 107.5 137.657257)
-		(end 110.5 137.657257)
-		(stroke
-			(width 0.5)
-			(type default)
-		)
-		(layer "Edge.Cuts")
-	)
-	(gr_circle
-		(center 107.68 22.657257)
-		(end 107.68 24.257257)
-		(stroke
-			(width 0.5)
-			(type default)
-		)
-		(fill no)
-		(layer "Edge.Cuts")
-	)
-	(gr_circle
-		(center 107.68 145.157257)
-		(end 107.68 146.757257)
-		(stroke
-			(width 0.5)
-			(type default)
-		)
-		(fill no)
-		(layer "Edge.Cuts")
-	)
-	(gr_line
-		(start 112.5 28.657257)
-		(end 115.5 28.657257)
-		(stroke
-			(width 0.5)
-			(type default)
-		)
-		(layer "Edge.Cuts")
-	)
-	(gr_line
-		(start 112.5 137.657257)
-		(end 115.5 137.657257)
-		(stroke
-			(width 0.5)
-			(type default)
-		)
-		(layer "Edge.Cuts")
-	)
-	(gr_circle
-		(center 114.64 22.657257)
-		(end 114.64 24.257257)
-		(stroke
-			(width 0.5)
-			(type default)
-		)
-		(fill no)
-		(layer "Edge.Cuts")
-	)
-	(gr_circle
-		(center 114.64 145.157257)
-		(end 114.64 146.757257)
-		(stroke
-			(width 0.5)
-			(type default)
-		)
-		(fill no)
-		(layer "Edge.Cuts")
-	)
-	(gr_line
-		(start 117.5 28.657257)
-		(end 120.5 28.657257)
-		(stroke
-			(width 0.5)
-			(type default)
-		)
-		(layer "Edge.Cuts")
-	)
-	(gr_line
-		(start 117.5 137.657257)
-		(end 120.5 137.657257)
-		(stroke
-			(width 0.5)
-			(type default)
-		)
-		(layer "Edge.Cuts")
-	)
 	(gr_rect
 		(start 123.5 33)
@@
 		(layer "Edge.Cuts")
 	)
-	(zone
-		(layer "F.Cu")
-		(hatch edge 0.5)
-		(connect_pads
-			(clearance 0.5)
-		)
-		(min_thickness 0.25)
-		(fill
-			(thermal_gap 0.5)
-			(thermal_bridge_width 0.5)
-			(island_removal_mode 0)
-		)
-		(polygon
-			(pts
-				(xy 101 19.657257) (xy 121.32 19.657257) (xy 121.32 148.157257) (xy 101 148.157257)
-			)
-		)
-	)
-	(zone
-		(layer "B.Cu")
-		(hatch edge 0.5)
-		(connect_pads
-			(clearance 0.5)
-		)
-		(min_thickness 0.25)
-		(fill
-			(thermal_gap 0.5)
-			(thermal_bridge_width 0.5)
-			(island_removal_mode 0)
-		)
-		(polygon
-			(pts
-				(xy 101 19.657257) (xy 121.32 19.657257) (xy 121.32 148.157257) (xy 101 148.157257)
-			)
-		)
-	)
 	(embedded_fonts no)
